Commit message: feat(So-101): make So-101/ a self-contained, git-tracked source of truth for robot geometry
- Re-generated So-101.urdf via scripts/mjcf_to_urdf.py against a fresh
  CoppeliaSim mesh export (arm .dae files) + the sim's vendored gripper
  STLs (So-101_gripper_*.stl, copied from
  LIBERO/libero/libero/assets/grippers/soarm_parallel/ since the old
  coppelia/ working directory was removed and never tracked in git)
- Updated scripts/mjcf_to_urdf.py's gripper mesh path constants to point
  at the new in-So-101/ filenames instead of the deleted ../coppelia/meshes/
  path, so the generator no longer depends on an external, untracked
  directory
- Renamed the fresh CoppeliaSim export's .dae files from the
  So-101-coppelia_* naming the export tool produced to the established
  bare So-101_* convention, so the generator script needed no changes
  for the arm meshes
- All 30 .dae arm meshes, 3 gripper STLs, and the whole-assembly
  So-101.stl/.obj/.mtl exports are now git-tracked (were previously
  untracked, which is exactly what let a manual deletion nearly lose
  the arm meshes with no recovery path)
- Verified: scripts/verify_urdf.py all-green, scripts/test_verify_urdf.py
  + LIBERO/libero/libero/envs/test_camera_config.py 7/7 pass

Co-Authored-By: Claude Sonnet 5 <noreply@anthropic.com>

File: So-101/So-101.urdf (robot description, URDF)
Before this commit: robot so101, 9 links, 8 joints
Links:
- link gripper_left_jaw: geometry collision box size=0.044 0.018 0.04; visual mesh filename=So-101_gripper_clamp_left_visual.stl scale=0.001 0.001 0.001
- link gripper_right_jaw: geometry collision box size=0.044 0.018 0.04; visual mesh filename=So-101_gripper_clamp_right_visual.stl scale=0.001 0.001 0.001
- link right_gripper: geometry visual mesh filename=So-101_gripper_main_frame_visual.stl scale=0.001 0.001 0.001
