Commit message: fix(quick-260919-h8v): regenerate URDF and update axis test expectations
- Regenerate So-101/So-101.urdf via scripts/mjcf_to_urdf.py from the
  Task-1-corrected MJCF: gripper_left axis 0 -1 0 -> 0 1 0, gripper_right
  axis 0 1 0 -> 0 -1 0, both limits 0..0.042 -> -0.042..0
- Update hardcoded expected axes in scripts/test_verify_urdf.py and
  scripts/verify_urdf.py to match
- Add 'from __future__ import annotations' to scripts/mjcf_to_urdf.py
  (Rule 3 blocking fix: the script's X | None type hints are Python 3.10+
  syntax, incompatible with the libero conda env's Python 3.9)
- Full TWIN-01..05 + env reset suite (7 tests) passes; verify_urdf.py CLI
  prints all checkmarks, no warnings

File: So-101/So-101.urdf (robot description, URDF)
Before this commit: robot so101, 9 links, 8 joints
Joints:
- joint gripper_left: axis 0 -1 0 -> 0 1 0; limit lower=0 upper=0.042 effort=60 velocity=0.5 -> lower=-0.042 upper=0 effort=60 velocity=0.5
- joint gripper_right: axis 0 1 0 -> 0 -1 0; limit lower=0 upper=0.042 effort=60 velocity=0.5 -> lower=-0.042 upper=0 effort=60 velocity=0.5

Commit message: fix(sim): establish Coppelia-aligned SO101 model and Phase 11 handoff

File: So-101/So-101.urdf (robot description, URDF)
Before this commit: robot so101, 9 links, 8 joints
Links:
- added link eef
- added link parallel_gripper_mechanism; visual cylinder length=0.01 radius=0.01; visual mesh filename=So-101_gripper_main_frame_visual.stl scale=0.001 0.001 0.001
- link right_gripper: geometry 
- link right_hand: geometry collision mesh filename=So-101_gripper_servo.stl; visual mesh filename=So-101_gripper_servo.stl
Joints:
- added joint gripper_mechanism_mount: type fixed, parent right_gripper, child parallel_gripper_mechanism, origin xyz=0.004443322423 0.000294707935691 0.000326451918819 rpy=-3.138416666 1.569999995 -3.089739806
- added joint gripper_to_eef: type fixed, parent right_gripper, child eef, origin xyz=-0.00161080382177 -0.000000415863769 -0.0766687457065 rpy=0 0 0
- joint gripper_left: limit lower=-0.042 upper=0 effort=60 velocity=0.5 -> lower=-0.036 upper=0 effort=60 velocity=0.5; parent right_gripper -> parallel_gripper_mechanism
- joint gripper_right: limit lower=-0.042 upper=0 effort=60 velocity=0.5 -> lower=-0.036 upper=0 effort=60 velocity=0.5; mimic (none) -> joint=gripper_left multiplier=1 offset=0; parent right_gripper -> parallel_gripper_mechanism

Commit message: fix(gripper): make increasing jaw position open the gripper

File: So-101/So-101.urdf (robot description, URDF)
Before this commit: robot so101, 11 links, 10 joints
Joints:
- joint gripper_left: axis 0 1 0 -> 0 -1 0; limit lower=-0.036 upper=0 effort=60 velocity=0.5 -> lower=0 upper=0.036 effort=60 velocity=0.5
- joint gripper_right: axis 0 -1 0 -> 0 1 0; limit lower=-0.036 upper=0 effort=60 velocity=0.5 -> lower=0 upper=0.036 effort=60 velocity=0.5
